File: Le_Tuto_Eclairant_HW/LTE_HW.kicad_pcb (KiCad board)
At the start: 2 copper layers, 45 x 74 mm, 10 parts, among them J1 Conn_01x03, SW1 SW_Push

Commit message: passage à kicad 6
Parts:
- RV1, RV2, RV3: value R_POT_Small -> R_Potentiometer_Small
- moved RV1 5.00 mm to (135.0, 139.0)
- moved RV2 5.00 mm to (135.0, 125.0)
- moved RV3 5.00 mm to (135.0, 111.0)
Connections:
- A1 pad 1: Net-(A1-Pad1) -> unconnected-(A1-Pad1)
- A1 pad 10: Net-(A1-Pad10) -> unconnected-(A1-Pad10)
- A1 pad 11: Net-(A1-Pad11) -> unconnected-(A1-Pad11)
- A1 pad 12: Net-(A1-Pad12) -> unconnected-(A1-Pad12)
- A1 pad 14: Net-(A1-Pad14) -> unconnected-(A1-Pad14)
- A1 pad 15: Net-(A1-Pad15) -> unconnected-(A1-Pad15)
- A1 pad 16: Net-(A1-Pad16) -> unconnected-(A1-Pad16)
- A1 pad 17: Net-(A1-Pad17) -> unconnected-(A1-Pad17)
- A1 pad 18: Net-(A1-Pad18) -> unconnected-(A1-Pad18)
- A1 pad 2: Net-(A1-Pad2) -> unconnected-(A1-Pad2)
- A1 pad 22: Net-(A1-Pad22) -> unconnected-(A1-Pad22)
- A1 pad 23: Net-(A1-Pad23) -> unconnected-(A1-Pad23)
- A1 pad 24: Net-(A1-Pad24) -> unconnected-(A1-Pad24)
- A1 pad 25: Net-(A1-Pad25) -> unconnected-(A1-Pad25)
- A1 pad 26: Net-(A1-Pad26) -> unconnected-(A1-Pad26)
- A1 pad 28: Net-(A1-Pad28) -> unconnected-(A1-Pad28)
- A1 pad 3: Net-(A1-Pad3) -> unconnected-(A1-Pad3)
- A1 pad 30: Net-(A1-Pad30) -> unconnected-(A1-Pad30)
- A1 pad 6: Net-(A1-Pad6) -> unconnected-(A1-Pad6)
- A1 pad 7: Net-(A1-Pad7) -> unconnected-(A1-Pad7)
- A1 pad 8: Net-(A1-Pad8) -> unconnected-(A1-Pad8)
- A1 pad 9: Net-(A1-Pad9) -> unconnected-(A1-Pad9)
Routing:
- net REF_5V: track 154.6 -> 152.6 mm
Other:
- net class Default removed
- net class fin removed
- net class gros removed
